File: hardware/v3s/power.sch (KiCad schematic (older format))
At the start: 33 parts, among them U2 AXP203

Commit message: working on ...
Parts:
- C1, C10, C11, C12, C13, C14, C15, C16, C17, C18, C19, C2, C21, C22, C23, C3, C6, C7, C8, C9: symbol X:C -> Device:C
- C4, C5: value 10uF -> 1uF; symbol X:C -> Device:C
- D1: value LED_Small -> CHGLED; symbol X:LED_Small -> Device:LED_Small
- L1, L2, L3: symbol X:L -> Device:L
- R4: renamed from R1; symbol X:R -> Device:R
- R5: renamed from R2; symbol X:R -> Device:R
- R6: renamed from R3; value 1K -> 200K; symbol X:R -> Device:R
- R7: renamed from R4; symbol X:R -> Device:R
- R8: renamed from R5; symbol X:R -> Device:R
Connections:
- wire segments 122 -> 130
