File: hardware/v3s/v3s.kicad_pcb (KiCad board)
At the start: 2 copper layers, 3 parts, among them U1 CY7C65213-32LTXI, U2 LNK403LG, U3 AT24CS32-STUM

Commit message: working on v3s
Parts:
- removed U2: LNK403LG, Power_Integrations:eSIP-7F
- removed U3: AT24CS32-STUM, TO_SOT_Packages_SMD:SOT-23-5
- U1: value CY7C65213-32LTXI -> V3S; footprint Housings_DFN_QFN:QFN-32-1EP_5x5mm_Pitch0.5mm -> Housings_QFP:LQFP-128_14x14mm_Pitch0.4mm
- moved U1 84.2 mm to (137.2, 74.9), turned to 45 degrees
Routing:
- net Net-(U1-Pad13): track 47.8 -> 0.00 mm
- net Net-(U1-Pad15): track 35.4 -> 0.00 mm, vias 1 -> 0
- net Net-(U1-Pad27): track 34.9 -> 0.00 mm

Commit message: working on v3s
Parts:
- added C1: 10uF, Capacitors_SMD:C_0603, F.Cu at (74.4, 51.9)
- added C10: 10uF, Capacitors_SMD:C_0603, F.Cu at (72.3, 62.0)
- added C11: 10uF, Capacitors_SMD:C_0603, F.Cu at (63.9, 63.0)
- added C12: 4.7uF, Capacitors_SMD:C_0603, F.Cu at (67.1, 56.9)
- added C13: 4.7uF, Capacitors_SMD:C_0603, F.Cu at (58.0, 69.0)
- added C14: 4.7uF, Capacitors_SMD:C_0603, F.Cu at (71.8, 56.9)
- added C15: 10uF, Capacitors_SMD:C_0603, F.Cu at (68.1, 62.0)
- added C16: 4.7uF, Capacitors_SMD:C_0603, F.Cu at (78.9, 51.9)
- added C17: 10uF, Capacitors_SMD:C_0603, F.Cu at (59.2, 57.9)
- added C18: 10uF, Capacitors_SMD:C_0603, F.Cu at (83.3, 51.9)
- added C19: 10uF/NC, Capacitors_SMD:C_0603, F.Cu at (55.1, 51.9)
- added C2: 10uF, Capacitors_SMD:C_0603, F.Cu at (68.1, 67.0)
- added C20: 10uF/NC, Capacitors_SMD:C_0603, F.Cu at (47.3, 67.6)
- added C21: 10uF, Capacitors_SMD:C_0603, F.Cu at (72.3, 67.0)
- added C22: 1uF, Capacitors_SMD:C_0603, F.Cu at (76.2, 62.0)
- added C23: 10uF, Capacitors_SMD:C_0603, F.Cu at (80.4, 56.9)
- added C3: 10uF, Capacitors_SMD:C_0603, F.Cu at (76.2, 56.9)
- added C4: 10uF, Capacitors_SMD:C_0603, F.Cu at (62.5, 68.0)
- added C5: 10uF, Capacitors_SMD:C_0603, F.Cu at (66.0, 51.9)
- added C6: 4.7uF, Capacitors_SMD:C_0603, F.Cu at (53.3, 69.0)
- added C7: 104, Capacitors_SMD:C_0603, F.Cu at (63.0, 57.9)
- added C8: 4.7uF, Capacitors_SMD:C_0603, F.Cu at (59.5, 63.0)
- added C9: 10uF, Capacitors_SMD:C_0603, F.Cu at (70.2, 51.9)
- added D1: LED_Small, Diodes_SMD:D_0603, F.Cu at (47.8, 62.6)
- added L1: 4.7uH, Pin_Headers:Pin_Header_Angled_1x02_Pitch1.00mm, F.Cu at (53.1, 56.9)
- added L2: 4.7uH, Pin_Headers:Pin_Header_Angled_1x02_Pitch1.00mm, F.Cu at (53.1, 63.0)
- added L3: 4.7uH, Pin_Headers:Pin_Header_Angled_1x02_Pitch1.00mm, F.Cu at (59.9, 51.9)
- added R1: 100R, Resistors_SMD:R_0402, F.Cu at (76.6, 66.9)
- added R2: 1K, Resistors_SMD:R_0402, F.Cu at (83.8, 56.8)
- added R3: 1K, Resistors_SMD:R_0402, F.Cu at (86.7, 51.7)
- added R4: 47K, Resistors_SMD:R_0402, F.Cu at (79.6, 61.8)
- added R5: 30mR, Resistors_SMD:R_0402, F.Cu at (62.6, 46.0)
- added U2: AXP203, Housings_DFN_QFN:UQFN-48-1EP_6x6mm_Pitch0.4mm, F.Cu at (54.5, 37.1)
- moved U1 72.4 mm to (75.1, 37.7), turned to 0 degrees

Commit message: working on ...
Parts:
- added R6: 200K, Resistors_SMD:R_0402, F.Cu at (82.6, 54.5)
- added R7: 47K, Resistors_SMD:R_0402, F.Cu at (69.5, 64.6)
- added R8: 30mR, Resistors_SMD:R_0402, F.Cu at (74.4, 59.5)
- C4, C5: value 10uF -> 1uF
- D1: value LED_Small -> CHGLED
- R1: value 100R -> R
- R2, R3: value 1K -> R
- R4: value 47K -> 100R
- R5: value 30mR -> 1K
- moved R2 49.2 mm to (37.0, 41.7)
- moved R3 48.6 mm to (38.2, 53.4)
- moved R1 47.1 mm to (35.5, 43.9)
- moved C6 28.8 mm to (68.5, 44.5)
- moved R5 25.9 mm to (88.5, 44.4)
- moved C20 25.1 mm to (57.3, 44.5)
- moved C18 22.4 mm to (61.0, 50.6)
- moved C2 20.7 mm to (79.3, 49.6)
- moved C5 17.0 mm to (81.4, 44.5)
- moved L1 15.4 mm to (62.2, 44.5)
- moved C22 14.2 mm to (83.1, 49.6)
- moved C8 13.8 mm to (65.4, 50.6)
- moved C21 13.8 mm to (78.3, 54.6)
- moved C14 13.6 mm to (77.4, 44.5)
- moved L2 13.5 mm to (54.9, 49.6)
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Connections:
- net DCDC2 renamed /power/DCDC2
- net Net-(U1-Pad67) renamed /cpu/DCDC2
- C22 pad 1: VBAT -> /power/VBAT
- C23 pad 1: VBAT -> /power/VBAT
- R1 pad 1: Net-(R1-Pad1) -> PS
- R1 pad 2: GND -> DCDC3
- R2 pad 1: Net-(D1-Pad2) -> PS
- R2 pad 2: /power/PS -> DCDC3
- R3 pad 1: Net-(R3-Pad1) -> PS
- R3 pad 2: GND -> DCDC3
- R4 pad 1: VCC-RTC -> Net-(R4-Pad1)
- R4 pad 2: /power/RESET -> GND
- R5 pad 1: VBAT -> Net-(D1-Pad2)
- R5 pad 2: Net-(C21-Pad1) -> /power/PS
- U1 pad 65: Net-(U1-Pad65) -> /cpu/VBAT
- U1 pad 66: Net-(U1-Pad66) -> /cpu/VBAT
- U1 pad 68: Net-(U1-Pad68) -> DCDC3
- U1 pad 69: Net-(U1-Pad69) -> PS
- U2 pad 23: Net-(R3-Pad1) -> Net-(R6-Pad1)
- U2 pad 37: Net-(R1-Pad1) -> Net-(R4-Pad1)
- U2 pad 38: VBAT -> /power/VBAT
- U2 pad 39: VBAT -> /power/VBAT
- U2 pad 42: VBAT -> /power/VBAT
- U2 pad 43: VBAT -> /power/VBAT
Routing:
- net PS: track 0.00 -> 20.5 mm
