File: hardware/v3s/v3s.sch (KiCad schematic (older format))
At the start: 4 parts, among them U1 CY7C65213-32LTXI, U2 LNK403LG, U3 AT24CS32-STUM, U4 UCC3800

Commit message: working on v3s
Parts:
- removed U1: CY7C65213-32LTXI, Housings_DFN_QFN:QFN-32-1EP_5x5mm_Pitch0.5mm, symbol cypress:CY7C65213-32LTXI
- removed U2: LNK403LG, Power_Integrations:eSIP-7F, symbol powerint:LNK403LG
- removed U3: AT24CS32-STUM, TO_SOT_Packages_SMD:SOT-23-5, symbol memory:AT24CS32-STUM
- removed U4: UCC3800, symbol ac-dc:UCC3800
- added U1: V3S, Housings_QFP:LQFP-128_14x14mm_Pitch0.4mm, symbol SOC_Allwinner_V3S:V3S
Connections:
- wire segments 14 -> 0
Changed lines of the file:
@@
 EESchema Schematic File Version 4
+LIBS:v3s-cache
 EELAYER 26 0
 EELAYER END
@@
 $EndDescr
 $Comp
-L powerint:LNK403LG U2
-U 1 1 5A3E7216
-P 5200 2950
-F 0 "U2" H 4870 2996 50  0000 R CNN
-F 1 "LNK403LG" H 4870 2905 50  0000 R CNN
-F 2 "Power_Integrations:eSIP-7F" H 5100 2950 50  0001 C CIN
-F 3 "http://www.powerint.com/sites/default/files/product-docs/linkswitch-ph_family_datasheet.pdf" H 5200 2950 50  0001 C CNN
-	1    5200 2950
+L SOC_Allwinner_V3S:V3S U1
+U 1 1 5A404065
+P 6000 3800
+F 0 "U1" H 8841 3921 50  0000 L CNN
+F 1 "V3S" H 8841 3830 50  0000 L CNN
+F 2 "Housings_QFP:LQFP-128_14x14mm_Pitch0.4mm" H 4850 3500 50  0001 C CNN
+F 3 "http://linux-sunxi.org/images/2/23/Allwinner_V3s_Datasheet_V1.0.pdf" H 4850 3500 50  0001 C CNN
+	1    6000 3800
 	1    0    0    -1
 $EndComp
-$Comp
-L cypress:CY7C65213-32LTXI U1
-U 1 1 5A3E72A5
-P 3650 3050
-F 0 "U1" H 3650 4028 50  0000 C CNN
-F 1 "CY7C65213-32LTXI" H 3650 3937 50  0000 C CNN
-F 2 "Housings_DFN_QFN:QFN-32-1EP_5x5mm_Pitch0.5mm" H 3650 1950 50  0001 C CNN
-F 3 "http://www.cypress.com/file/139881/download" H 1150 3550 50  0001 C CNN
-	1    3650 3050
-	1    0    0    -1
-$EndComp
-Wire Wire Line
-	4250 2450 5000 2450
-Wire Wire Line
-	5000 2450 5000 2650
-Wire Wire Line
-	4250 2550 5300 2550
-Wire Wire Line
-	5300 2550 5300 2650
-Wire Wire Line
-	4250 2750 4700 2750
-Wire Wire Line
-	4700 2750 4700 3300
-Wire Wire Line
-	4700 3300 5000 3300
-Wire Wire Line
-	5000 3300 5000 3250
-Wire Wire Line
-	5200 3250 5200 3450
-Wire Wire Line
-	5200 3450 4250 3450
-Wire Wire Line
-	5400 3250 5400 3650
-Wire Wire Line
-	5400 3650 4250 3650
-Wire Wire Line
-	5600 2950 5600 3850
-Wire Wire Line
-	5600 3850 4250 3850
-$Comp
-L ac-dc:UCC3800 U4
-U 1 1 5A3E75E2
-P 6550 1800
-F 0 "U4" H 6550 2378 50  0000 C CNN
-F 1 "UCC3800" H 6550 2287 50  0000 C CNN
-F 2 "" H 6550 1800 50  0001 C CNN
-F 3 "http://www.ti.com/lit/ds/symlink/ucc3800.pdf" H 6550 1800 50  0001 C CNN
-	1    6550 1800
-	1    0    0    -1
-$EndComp
-$Comp
-L memory:AT24CS32-STUM U3
-U 1 1 5A3E79CE
-P 4900 1800
-F 0 "U3" H 4900 2328 50  0000 C CNN
-F 1 "AT24CS32-STUM" H 4900 2237 50  0000 C CNN
-F 2 "TO_SOT_Packages_SMD:SOT-23-5" H 4900 1800 50  0001 C CIN
-F 3 "http://www.atmel.com/Images/Atmel-8869-SEEPROM-AT24CS32-Datasheet.pdf" H 4900 1800 50  0001 C CNN
-	1    4900 1800
-	1    0    0    -1
-$EndComp

Commit message: working on v3s
Parts:
- removed U1: V3S, Housings_QFP:LQFP-128_14x14mm_Pitch0.4mm, symbol SOC_Allwinner_V3S:V3S
- added U?: V3S, symbol x:V3S
Changed lines of the file:
@@
 $EndDescr
 $Comp
-L SOC_Allwinner_V3S:V3S U1
-U 1 1 5A404065
-P 6000 3800
-F 0 "U1" H 8841 3921 50  0000 L CNN
-F 1 "V3S" H 8841 3830 50  0000 L CNN
-F 2 "Housings_QFP:LQFP-128_14x14mm_Pitch0.4mm" H 4850 3500 50  0001 C CNN
-F 3 "http://linux-sunxi.org/images/2/23/Allwinner_V3s_Datasheet_V1.0.pdf" H 4850 3500 50  0001 C CNN
-	1    6000 3800
+L x:V3S U?
+U 1 1 5A3ED1F1
+P 5850 3700
+F 0 "U?" H 8691 3775 50  0000 L CNN
+F 1 "V3S" H 6150 3900 50  0001 C CNN
+F 2 "" H 4700 3400 50  0001 C CNN
+F 3 "http://linux-sunxi.org/images/2/23/Allwinner_V3s_Datasheet_V1.0.pdf" H 4700 3400 50  0001 C CNN
+	1    5850 3700
 	1    0    0    -1
 $EndComp

Commit message: working on v3s
Parts:
- removed U?: V3S, symbol x:V3S
Changed lines of the file:
@@
 $Descr A4 11693 8268
 encoding utf-8
-Sheet 1 1
+Sheet 1 3
 Title ""
 Date ""
@@
 Comment4 ""
 $EndDescr
-$Comp
-L x:V3S U?
-U 1 1 5A3ED1F1
-P 5850 3700
-F 0 "U?" H 8691 3775 50  0000 L CNN
-F 1 "V3S" H 6150 3900 50  0001 C CNN
-F 2 "" H 4700 3400 50  0001 C CNN
-F 3 "http://linux-sunxi.org/images/2/23/Allwinner_V3s_Datasheet_V1.0.pdf" H 4700 3400 50  0001 C CNN
-	1    5850 3700
-	1    0    0    -1
-$EndComp
+$Sheet
+S 850  850  1550 1300
+U 5A4181B4
+F0 "cpu" 50
+F1 "cpu.sch" 50
+$EndSheet
+$Sheet
+S 2650 850  1500 1300
+U 5A4181BB
+F0 "power" 50
+F1 "power.sch" 50
+$EndSheet
 $EndSCHEMATC

Commit message: working on ...
Changed lines of the file:
@@
 $Descr A4 11693 8268
 encoding utf-8
-Sheet 1 3
+Sheet 1 4
 Title ""
 Date ""
@@
 F1 "power.sch" 50
 $EndSheet
+$Sheet
+S 4450 850  1300 1300
+U 5A535D2D
+F0 "spinor" 50
+F1 "spinor.sch" 50
+$EndSheet
 $EndSCHEMATC
